File: Hardware/Schematic.sch (EAGLE design)
At the start: 105 parts, among them IC1 DRV2605YZFR_DRV2605YZFR, IC2 BQ25180YBGR_BQ25180YBGR, IC3 BMA423_BMA423, IC9 RT6160AWSC_RT6160AWSC, J1 503480-2400_503480-2400, J2 TC2030-IDC_TC2030-IDC, J4 KH-TYPE-C-16P_KH-TYPE-C-16P, Q3 ESP32_C6_LIBRARY_6_SI1308EDL-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, U1 NORDIC_NRF_4_NRF52840_QF, U3 ESP32_C6_LIBRARY_MAX17048G+T10, X2 32.768kHz

Commit message: Rename nets for clarity and consistency
Connections:
- net N$127 renamed EPD_OP
- net N$128 renamed EPD_ON
- net N$13 renamed VREG
- net N$137 renamed VBAT
- net N$19 renamed I2C_SCL
- net N$20 renamed I2C_SDA
- net N$33 renamed VDD_3V3_MON
- net N$34 renamed NRST
- net N$35 renamed SWDCLK
- net N$36 renamed SWDIO
- net N$37 renamed SWO
- net N$74 renamed RF_MCU_MATCH
- net N$75 renamed RF_MATCH_ANT
- net N$9 renamed VDD_3V3
Changed lines of the file:
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@@
 </segment>
 </net>
-<net name="N$9" class="0">
+<net name="VDD_3V3" class="0">
 <segment>
 <pinref part="TP_3V3" gate="G$1" pin="TP"/>
@@
 </segment>
 </net>
-<net name="N$13" class="0">
+<net name="VREG" class="0">
 <segment>
 <pinref part="TP_VREG" gate="G$1" pin="TP"/>
@@
 </segment>
 </net>
-<net name="N$19" class="0">
+<net name="I2C_SCL" class="0">
 <segment>
 <pinref part="TP_SCL" gate="G$1" pin="TP"/>
@@
 </segment>
 </net>
-<net name="N$20" class="0">
+<net name="I2C_SDA" class="0">
 <segment>
 <pinref part="TP_SDA" gate="G$1" pin="TP"/>
@@
 </segment>
 </net>
-<net name="N$33" class="0">
+<net name="VDD_3V3_MON" class="0">
 <segment>
 <pinref part="TP_3.3V" gate="G$1" pin="TP"/>
@@
 </segment>
 </net>
-<net name="N$34" class="0">
+<net name="NRST" class="0">
 <segment>
 <pinref part="TP_RESET" gate="G$1" pin="TP"/>
@@
 </segment>
 </net>
-<net name="N$35" class="0">
+<net name="SWDCLK" class="0">
 <segment>
 <pinref part="TP_SWDCLK" gate="G$1" pin="TP"/>
@@
 </segment>
 </net>
-<net name="N$36" class="0">
+<net name="SWDIO" class="0">
 <segment>
 <pinref part="TP_SWDIO" gate="G$1" pin="TP"/>
@@
 </segment>
 </net>
-<net name="N$37" class="0">
+<net name="SWO" class="0">
 <segment>
 <pinref part="TP_SWO" gate="G$1" pin="TP"/>
@@
 </segment>
 </net>
-<net name="N$74" class="0">
+<net name="RF_MCU_MATCH" class="0">
 <segment>
 <pinref part="U1" gate="G$1" pin="ANT@H23"/>
@@
 </segment>
 </net>
-<net name="N$75" class="0">
+<net name="RF_MATCH_ANT" class="0">
 <segment>
 <pinref part="L1" gate="L$1" pin="2"/>
@@
 </segment>
 </net>
-<net name="N$127" class="0">
+<net name="EPD_OP" class="0">
 <segment>
 <pinref part="TP_OP" gate="G$1" pin="TP"/>
@@
 </segment>
 </net>
-<net name="N$128" class="0">
+<net name="EPD_ON" class="0">
 <segment>
 <pinref part="TP_ON" gate="G$1" pin="TP"/>
@@
 </segment>
 </net>
-<net name="N$137" class="0">
+<net name="VBAT" class="0">
 <segment>
 <pinref part="TP_VBAT" gate="G$1" pin="TP"/>
